Commit message: Adapting constructor files to our package

File: hc10_kinect_description/urdf/hc10.xacro (robot description, xacro)
@@ -1,5 +1,5 @@
 <?xml version="1.0" ?>
 <robot name="motoman_hc10" xmlns:xacro="http://ros.org/wiki/xacro">
-  <xacro:include filename="$(find motoman_hc10_support)/urdf/hc10_macro.xacro" />
+  <xacro:include filename="$(find hc10_kinect_description)/urdf/hc10_macro.xacro" />
   <xacro:motoman_hc10 prefix=""/>
 </robot>

File: hc10_kinect_description/urdf/hc10_macro.xacro (robot description, xacro)
@@ -8,11 +8,11 @@
       <visual>
         <geometry>
-          <mesh filename="package://motoman_hc10_support/meshes/hc10/visual/base_link.dae"/>
-        </geometry>
-        <xacro:material_yaskawa_blue/>
-      </visual>
-      <collision>
-        <geometry>
-          <mesh filename="package://motoman_hc10_support/meshes/hc10/collision/base_link.stl"/>
+          <mesh filename="package://hc10_kinect_description/meshes/visual/base_link.dae"/>
+        </geometry>
+        <xacro:material_yaskawa_blue/>
+      </visual>
+      <collision>
+        <geometry>
+          <mesh filename="package://hc10_kinect_description/meshes/collision/base_link.stl"/>
         </geometry>
       </collision>
@@ -26,11 +26,11 @@
       <visual>
         <geometry>
-          <mesh filename="package://motoman_hc10_support/meshes/hc10/visual/link_1_s.dae"/>
-        </geometry>
-        <xacro:material_yaskawa_blue/>
-      </visual>
-      <collision>
-        <geometry>
-          <mesh filename="package://motoman_hc10_support/meshes/hc10/collision/link_1_s.stl"/>
+          <mesh filename="package://hc10_kinect_description/meshes/visual/link_1_s.dae"/>
+        </geometry>
+        <xacro:material_yaskawa_blue/>
+      </visual>
+      <collision>
+        <geometry>
+          <mesh filename="package://hc10_kinect_description/meshes/collision/link_1_s.stl"/>
         </geometry>
       </collision>
@@ -44,11 +44,11 @@
       <visual>
         <geometry>
-          <mesh filename="package://motoman_hc10_support/meshes/hc10/visual/link_2_l.dae"/>
-        </geometry>
-        <xacro:material_yaskawa_blue/>
-      </visual>
-      <collision>
-        <geometry>
-          <mesh filename="package://motoman_hc10_support/meshes/hc10/collision/link_2_l.stl"/>
+          <mesh filename="package://hc10_kinect_description/meshes/visual/link_2_l.dae"/>
+        </geometry>
+        <xacro:material_yaskawa_blue/>
+      </visual>
+      <collision>
+        <geometry>
+          <mesh filename="package://hc10_kinect_description/meshes/collision/link_2_l.stl"/>
         </geometry>
       </collision>
@@ -62,11 +62,11 @@
       <visual>
         <geometry>
-          <mesh filename="package://motoman_hc10_support/meshes/hc10/visual/link_3_u.dae"/>
-        </geometry>
-        <xacro:material_yaskawa_blue/>
-      </visual>
-      <collision>
-        <geometry>
-          <mesh filename="package://motoman_hc10_support/meshes/hc10/collision/link_3_u.stl"/>
+          <mesh filename="package://hc10_kinect_description/meshes/visual/link_3_u.dae"/>
+        </geometry>
+        <xacro:material_yaskawa_blue/>
+      </visual>
+      <collision>
+        <geometry>
+          <mesh filename="package://hc10_kinect_description/meshes/collision/link_3_u.stl"/>
         </geometry>
       </collision>
@@ -80,11 +80,11 @@
       <visual>
         <geometry>
-          <mesh filename="package://motoman_hc10_support/meshes/hc10/visual/link_4_r.dae"/>
-        </geometry>
-        <xacro:material_yaskawa_blue/>
-      </visual>
-      <collision>
-        <geometry>
-          <mesh filename="package://motoman_hc10_support/meshes/hc10/collision/link_4_r.stl"/>
+          <mesh filename="package://hc10_kinect_description/meshes/visual/link_4_r.dae"/>
+        </geometry>
+        <xacro:material_yaskawa_blue/>
+      </visual>
+      <collision>
+        <geometry>
+          <mesh filename="package://hc10_kinect_description/meshes/collision/link_4_r.stl"/>
         </geometry>
       </collision>
@@ -98,11 +98,11 @@
       <visual>
         <geometry>
-          <mesh filename="package://motoman_hc10_support/meshes/hc10/visual/link_5_b.dae"/>
-        </geometry>
-        <xacro:material_yaskawa_blue/>
-      </visual>
-      <collision>
-        <geometry>
-          <mesh filename="package://motoman_hc10_support/meshes/hc10/collision/link_5_b.stl"/>
+          <mesh filename="package://hc10_kinect_description/meshes/visual/link_5_b.dae"/>
+        </geometry>
+        <xacro:material_yaskawa_blue/>
+      </visual>
+      <collision>
+        <geometry>
+          <mesh filename="package://hc10_kinect_description/meshes/collision/link_5_b.stl"/>
         </geometry>
       </collision>
@@ -116,11 +116,11 @@
       <visual>
         <geometry>
-          <mesh filename="package://motoman_hc10_support/meshes/hc10/visual/link_6_t.dae"/>
-        </geometry>
-        <xacro:material_yaskawa_blue/>
-      </visual>
-      <collision>
-        <geometry>
-          <mesh filename="package://motoman_hc10_support/meshes/hc10/collision/link_6_t.stl"/>
+          <mesh filename="package://hc10_kinect_description/meshes/visual/link_6_t.dae"/>
+        </geometry>
+        <xacro:material_yaskawa_blue/>
+      </visual>
+      <collision>
+        <geometry>
+          <mesh filename="package://hc10_kinect_description/meshes/collision/link_6_t.stl"/>
         </geometry>
       </collision>
