Commit message: ajout modif reglage nuage de point

File: hc10_kinect_description/urdf/camera.xacro (robot description, xacro)
@@ -24,5 +24,5 @@
     <link name="kinect_link_optical"></link>
      <joint name="kinect_optical_joint" type="fixed">
-        <origin xyz="0 0 0" rpy="0 0 0" />
+        <origin xyz="0 0 0" rpy="${-pi/2} 0  ${-pi/2}" />
         <parent link="kinect_link" />
         <child link="kinect_link_optical" />
