Commit message: adding octomap

File: hc10_kinect_description/urdf/hc10_macro.xacro (robot description, xacro)
@@ -133,5 +133,5 @@
     <!-- end of link list -->
     <!-- joint list -->
-    <joint name="world_fixed" type="fixed">
+    <joint name="map_fixed" type="fixed">
       <parent link="world"/>
       <child link="${prefix}base_link"/>

Commit message: Adding Inverse Kinematics solver

File: hc10_kinect_description/urdf/hc10_macro.xacro (robot description, xacro)
@@ -2,4 +2,19 @@
 <robot xmlns:xacro="http://ros.org/wiki/xacro">
   <xacro:macro name="motoman_hc10" params="prefix">
+    <material name="white">
+      <color rgba="1 1 1 1"/>
+    </material>
+    <material name="orange">
+      <color rgba="1 0.3 0.1 1"/>
+    </material>
+    <material name="blue">
+      <color rgba="0.2 0.2 1 1"/>
+    </material>
+    <material name="red">
+      <color rgba="1 0 0 1"/>
+    </material>
+    <material name="black">
+      <color rgba="0 0 0 1"/>
+    </material>
     <!-- link list -->
     <link name="world"/>
