Commit message: Adding sensor in sumulation

File: hc10_kinect_moveit_config/config/gazebo_motoman_hc10.urdf (robot description, URDF)
Before this commit: robot motoman_hc10, 10 links, 9 joints
Links:
- added link kinect_link; collision box size=0.2 0.05 0.05; visual box size=0.2 0.05 0.05
Joints:
- added joint kinect_joint: type fixed, parent tool0, child kinect_link, origin xyz=0 0 0.03 rpy=0 0 0
